File: design_files/LaserBoard.kicad_sch (KiCad schematic)
At the start: 11 parts, among them J12 RJ45_Amphenol_RJMG1BD3B8K1ANR, J13 Conn_01x06, J14 Conn_01x02_Pin, J15 Conn_01x03, U1 Teensy4.1

Commit message: And that's why we write documentation - two small errors on the pcb
Connections:
- net +5V: now also JP12.2 (C), U1.48 (VIN); no longer JP12.3 (B)
- new net 5V_SUPPLY: JP12.3 (B)
Changed lines of the file:
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@@
   (junction (at 215.392 137.414) (diameter 0) (color 0 0 0 0)
+  )
+  (junction (at 198.374 45.339) (diameter 0) (color 0 0 0 0)
   )
   (junction (at 219.202 137.414) (diameter 0) (color 0 0 0 0)
@@
     (stroke (width 0) (type default))
   )
-  (wire (pts (xy 198.374 47.498) (xy 198.374 40.132))
+  (wire (pts (xy 198.374 47.498) (xy 198.374 45.339))
     (stroke (width 0) (type default))
   )
@@
     (stroke (width 0) (type default))
   )
+  (wire (pts (xy 198.374 45.339) (xy 198.374 40.132))
+    (stroke (width 0) (type default))
+  )
   (wire (pts (xy 119.126 57.658) (xy 133.096 57.658))
     (stroke (width 0) (type default))
@@
   )
   (wire (pts (xy 192.532 80.518) (xy 192.532 83.058))
+    (stroke (width 0) (type default))
+  )
+  (wire (pts (xy 198.374 45.339) (xy 200.787 45.339))
     (stroke (width 0) (type default))
   )
@@
   (label "R+" (at 192.278 124.968 0) (fields_autoplaced)
     (effects (font (size 1.27 1.27)) (justify left bottom))
+  )
+  (global_label "5V_SUPPLY" (shape input) (at 203.454 34.29 90) (fields_autoplaced)
+    (effects (font (size 1.27 1.27)) (justify left))
+    (property "Intersheetrefs" "${INTERSHEET_REFS}" (at 203.454 20.9218 90)
+      (effects (font (size 1.27 1.27)) (justify left) hide)
+    )
   )
   (global_label "PWR_5" (shape input) (at 133.096 98.298 180) (fields_autoplaced)
@@
     )
   )
-  (symbol (lib_id "power:+5V") (at 203.454 34.29 0) (unit 1)
+  (symbol (lib_id "power:+5V") (at 200.787 45.339 270) (unit 1)
     (in_bom yes) (on_board yes) (dnp no) (fields_autoplaced)
-    (property "Reference" "#PWR055" (at 203.454 38.1 0)
-      (effects (font (size 1.27 1.27)) hide)
-    )
-    (property "Value" "+5V" (at 203.454 30.988 0)
-      (effects (font (size 1.27 1.27)))
-    )
-    (property "Footprint" "" (at 203.454 34.29 0)
-      (effects (font (size 1.27 1.27)) hide)
-    )
-    (property "Datasheet" "" (at 203.454 34.29 0)
-      (effects (font (size 1.27 1.27)) hide)
-    )
+    (property "Reference" "#PWR055" (at 196.977 45.339 0)
+      (effects (font (size 1.27 1.27)) hide)
+    )
+    (property "Value" "+5V" (at 204.089 45.974 90)
+      (effects (font (size 1.27 1.27)) (justify left))
+    )
+    (property "Footprint" "" (at 200.787 45.339 0)
+      (effects (font (size 1.27 1.27)) hide)
+    )
+    (property "Datasheet" "" (at 200.787 45.339 0)
+      (effects (font (size 1.27 1.27)) hide)
+    )

Commit message: BOM, readme update
Parts:
- C12: value 0.1uF, 16V -> 0.1uF, 50V; MouserPN (none) -> 80-C603C104K5RAC3121; mpn (none) -> C603C104K5RAC3121
- J12: MouserPN (none) -> 710-618015231321; mpn (none) -> 618015231321
- JP12: value SolderJumper_3_Open -> Jumper 3 Position, Open
Changed lines of the file:
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@@
       (effects (font (size 1.27 1.27)))
     )
-    (property "Value" "SolderJumper_3_Open" (at 198.374 34.29 0)
+    (property "Value" "Jumper 3 Position, Open" (at 198.374 34.29 0)
       (effects (font (size 1.27 1.27)) hide)
     )
@@
     )
     (property "Datasheet" "https://www.amphenolcanada.com/ProductSearch/Drawings/AC/RJMG1BD3B8K1ANR.PDF" (at 245.11 101.854 0)
+      (effects (font (size 1.27 1.27)) hide)
+    )
+    (property "MouserPN" "710-618015231321" (at 245.11 122.174 0)
+      (effects (font (size 1.27 1.27)) hide)
+    )
+    (property "mpn" "618015231321" (at 245.11 122.174 0)
       (effects (font (size 1.27 1.27)) hide)
     )
@@
       (effects (font (size 1.27 1.27)) (justify left))
     )
-    (property "Value" "0.1uF, 16V" (at 214.63 135.509 0)
+    (property "Value" "0.1uF, 50V" (at 214.63 135.509 0)
       (effects (font (size 1.27 1.27)) (justify left))
     )
@@
       (effects (font (size 1.27 1.27)) hide)
     )
+    (property "MouserPN" "80-C603C104K5RAC3121" (at 211.074 133.604 0)
+      (effects (font (size 1.27 1.27)) hide)
+    )
+    (property "mpn" "C603C104K5RAC3121" (at 211.074 133.604 0)
+      (effects (font (size 1.27 1.27)) hide)
+    )

Commit message: Rev 5a
Parts:
- U1: Notes (none) -> Don't purchase from Mouser - export control paperwork is sl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
Connections:
- net GND: now also C12.1, J12.L1 (LEDY_A); no longer C12.2, J12.L3 (LEDG_K)
- net at J12.L2 (LEDY_K): now also U1.61 (LED)
- net at J12.L4 (LEDG_A): no longer U1.61 (LED)
- net at J12.R2 (TCT), J12.R5 (RCT): now also C12.2; no longer C12.1
Other:
- moved on the sheet: C12
