File: design_files/MotorIO.kicad_sch (KiCad schematic)
At the start: 59 parts, among them J1 Conn_01x03_Socket, J2 Conn_01x03_Socket, J3 Conn_01x03_Socket, J4 Conn_01x03_Socket, J5 Conn_01x02_Socket, J6 Conn_01x04_Socket, J7 Conn_01x04_Socket, J8 Conn_01x04_Socket, J9 Conn_01x04_Socket, U3 74HC245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

Commit message: BOM, readme update
Parts:
- C1, C7: value 0.1uF, 16V -> 0.1uF, 25V; MouserPN (none) -> 187-CL05A104KA5NNNC; mpn (none) -> CL05A104KA5NNNC
- C2, C3, C4, C5, C6: mpn (none) -> CGA3E1X7R1C105AC
- D1, D10, D2, D3, D4, D5, D6, D7, D8: mpn (none) -> 1N4148W-F
- D11, D12, D13, D14: mpn (none) -> 150060GS75000
- D9: mpn (none) -> 150060RS75000
- J1, J2, J3, J4: value Conn_01x03_Socket -> Type KK 1x03 Socket; mpn (none) -> 61900311121
- J5: value Conn_01x02_Socket -> Type KK 1x02 Socket; mpn (none) -> 61900211121
- J6, J7, J8, J9: value Conn_01x04_Socket -> Type KK 1x04 Socket; mpn (none) -> 61900411121
- JP1, JP2, JP3, JP4, JP5, JP6, JP7, JP8: value Jumper_2_Open -> Jumper 2 Position, Open
- U3, U4: MouserPN (none) -> 771-74AHC245PW-Q100J; mpn (none) -> 74AHC245PW-Q100J
Connections:
- net +5V: now also J5.1 (Pin_1); no longer J5.2 (Pin_2)
- net at R15.1: now also J5.2 (Pin_2); no longer J5.1 (Pin_1)
Other:
- moved on the sheet: J5

Commit message: Rev 5a
Parts:
- removed JP3, JP5, JP7: Jumper 2 Position, Open, LaserBoardR5:SolderJumper-2_P1.3mm_Open_RoundedPad1.0x1.5mm, symbol LaserBoardR5:Jumper_2_Open
- added JP14, JP15, JP17, JP19, JP21, JP3, JP5, JP7: Jumper_2_Bridged, LaserBoardR5:SolderJumper-2_P1.3mm_Bridged_RoundedPad1.0x1.5mm, symbol Jumper:Jumper_2_Bridged
- added JP16, JP18, JP20: Jumper 2 Position, Open, LaserBoardR5:SolderJumper-2_P1.3mm_Open_RoundedPad1.0x1.5mm, symbol LaserBoardR5:Jumper_2_Open
- C1, C7: Notes (none) -> Generic decoupling cap
- R1, R10, R11, R12, R14, R15, R2, R3, R4, R5, R6, R7, R8, R9: MouserPN (none) -> 603-RC0603JR-0710KL; mpn (none) -> RC0603JR-0710KL
- R13, R16, R17, R18, R19: MouserPN (none) -> 603-RC0603JR-0720KL; mpn (none) -> RC0603JR-0720KL
Connections:
- net +5V: now also JP14.1 (A), JP3.1 (A), JP5.1 (A), JP7.1 (A); no longer JP1.2 (B)
- net at R4.1: now also JP3.2 (B)
- net at D3.2 (A), R4.2: now also JP17.1 (A)
- net at D8.1 (K), R10.2: now also JP20.1 (A)
- net at J1.2 (Pin_2), R1.1: now also JP1.2 (B), JP15.2 (B)
- net at D1.2 (A), R2.2: now also JP15.1 (A)
- net at D6.1 (K), R8.2: now also JP18.1 (A)
- net at R9.1: now also JP7.2 (B)
- net at R2.1: now also JP14.2 (B); no longer JP1.1 (A)
- net at J3.2 (Pin_2), R11.1: now also JP18.2 (B), JP19.2 (B)
- net at J2.2 (Pin_2), R6.1: now also JP16.2 (B), JP17.2 (B)
- net at D4.1 (K), R5.2: now also JP16.1 (A)
- net at D7.2 (A), R9.2: now also JP21.1 (A)
- net at J4.2 (Pin_2), R12.1: now also JP20.2 (B), JP21.2 (B)
- net at D10.1 (K), R14.2: now also J5.2 (Pin_2), R15.1
- net at D2.1 (K), R3.2: now also JP1.1 (A)
- net at R7.1: now also JP5.2 (B)
- net at D5.2 (A), R7.2: now also JP19.1 (A)
Other:
- note removed: "Limit 1"
- note removed: "Limit 2"
- note removed: "Limit 3"
- moved on the sheet: D1, D2, J1, JP1, JP2, R1, R2, R3
