File: design_files/PowerSupply.kicad_sch (KiCad schematic)
At the start: 16 parts, among them J17 Screw_Terminal_01x02, J18 Screw_Terminal_01x02, U9 VX7805-500

Commit message: And that's why we write documentation - two small errors on the pcb
Connections:
- net +5V renamed 5V_SUPPLY
Changed lines of the file:
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@@
+    )
+  )
+  (global_label "5V_SUPPLY" (shape input) (at 119.634 151.638 90) (fields_autoplaced)
+    (effects (font (size 1.27 1.27)) (justify left))
+    (property "Intersheetrefs" "${INTERSHEET_REFS}" (at 119.634 138.2698 90)
+      (effects (font (size 1.27 1.27)) (justify left) hide)
     )
   )
@@
         )
       )
-    )
-  )
-  (symbol (lib_id "power:+5V") (at 119.634 151.638 0) (unit 1)
-    (in_bom yes) (on_board yes) (dnp no) (fields_autoplaced)
-    (property "Reference" "#PWR062" (at 119.634 155.448 0)
-      (effects (font (size 1.27 1.27)) hide)
-    )
-    (property "Value" "+5V" (at 119.634 148.336 0)
-      (effects (font (size 1.27 1.27)))
-    )
-    (property "Footprint" "" (at 119.634 151.638 0)
-      (effects (font (size 1.27 1.27)) hide)
-    )
-    (property "Datasheet" "" (at 119.634 151.638 0)
-      (effects (font (size 1.27 1.27)) hide)
-    )
-    (pin "1")
-    (instances
-      (project "LaserBoard"
-        (path "/4d77737b-9eff-481f-ac50-cf5a7c761856/fd615519-c9a1-4056-80cd-d13305f563e0"
-          (reference "#PWR062") (unit 1)
-        )
-      )

Commit message: BOM, readme update
Parts:
- C13, C14: footprint LaserBoardR5:C_0603_1608Metric_Pad1.08x0.95mm_HandSolder -> LaserBoardR5:C_0603_1608Metric; mpn (none) -> C603C104K5RAC3121
- C16, C18: mpn (none) -> CL32A106KAULNNE
- C17: mpn (none) -> CL21A475KLCLQNC
- D16, D17: mpn (none) -> 150060GS75000
- FB1: MouserPN (none) -> 81-BLM41P600S; mpn (none) -> BLM41PG600SN1L
Connections:
- net GND: now also J18.2 (Pin_2); no longer J18.1 (Pin_1)
- net V_INPUT: now also J18.1 (Pin_1); no longer J18.2 (Pin_2)
Changed lines of the file:
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@@
   (junction (at 101.6 170.688) (diameter 0) (color 0 0 0 0)
   )
+  (junction (at 90.678 96.012) (diameter 0) (color 0 0 0 0)
+  )
   (junction (at 154.686 94.234) (diameter 0) (color 0 0 0 0)
   )
@@
     (stroke (width 0) (type default))
   )
+  (wire (pts (xy 88.519 94.234) (xy 88.519 91.694))
+    (stroke (width 0) (type default))
+  )
   (wire (pts (xy 41.91 151.384) (xy 41.91 153.924))
     (stroke (width 0) (type default))
   )
+  (wire (pts (xy 90.678 96.012) (xy 90.678 99.314))
+    (stroke (width 0) (type default))
+  )
   (wire (pts (xy 138.176 75.946) (xy 143.002 75.946))
     (stroke (width 0) (type default))
@@
     (stroke (width 0) (type default))
   )
+  (wire (pts (xy 83.82 94.234) (xy 88.519 94.234))
+    (stroke (width 0) (type default))
+  )
   (wire (pts (xy 48.514 153.924) (xy 48.514 155.702))
     (stroke (width 0) (type default))
@@
     (stroke (width 0) (type default))
   )
+  (wire (pts (xy 83.82 91.694) (xy 86.487 91.694))
+    (stroke (width 0) (type default))
+  )
   (wire (pts (xy 154.686 75.946) (xy 167.386 75.946))
     (stroke (width 0) (type default))
@@
     (stroke (width 0) (type default))
   )
-  (wire (pts (xy 91.694 91.694) (xy 83.82 91.694))
-    (stroke (width 0) (type default))
-  )
   (wire (pts (xy 101.6 153.67) (xy 119.634 153.67))
     (stroke (width 0) (type default))
@@
     (stroke (width 0) (type default))
   )
+  (wire (pts (xy 88.519 91.694) (xy 91.694 91.694))
+    (stroke (width 0) (type default))
+  )
   (wire (pts (xy 119.634 153.67) (xy 119.634 153.924))
     (stroke (width 0) (type default))
@@
     (stroke (width 0) (type default))
   )
-  (wire (pts (xy 90.678 94.234) (xy 90.678 99.314))
+  (wire (pts (xy 90.678 94.234) (xy 90.678 96.012))
     (stroke (width 0) (type default))
   )
@@
     (stroke (width 0) (type default))
   )
-  (wire (pts (xy 90.678 94.234) (xy 83.82 94.234))
-    (stroke (width 0) (type default))
-  )
   (wire (pts (xy 143.002 91.948) (xy 143.002 94.234))
     (stroke (width 0) (type default))
@@
   )
   (wire (pts (xy 83.82 170.688) (xy 83.82 173.736))
+    (stroke (width 0) (type default))
+  )
+  (wire (pts (xy 86.487 96.012) (xy 90.678 96.012))
+    (stroke (width 0) (type default))
+  )
+  (wire (pts (xy 86.487 91.694) (xy 86.487 96.012))
     (stroke (width 0) (type default))
   )
@@
       (effects (font (size 1.27 1.27)) (justify left))
     )
-    (property "Footprint" "LaserBoardR5:C_0603_1608Metric_Pad1.08x0.95mm_HandSolder" (at 127.2032 91.694 0)
+    (property "Footprint" "LaserBoardR5:C_0603_1608Metric" (at 127.2032 91.694 0)
       (effects (font (size 1.27 1.27)) hide)
     )
@@
     )
     (property "MouserPN" "80-C603C104K5RAC3121" (at 126.238 87.884 0)
+      (effects (font (size 1.27 1.27)) hide)
+    )
+    (property "mpn" "C603C104K5RAC3121" (at 126.238 87.884 0)
       (effects (font (size 1.27 1.27)) hide)
     )
@@
       (effects (font (size 1.27 1.27)) hide)
     )
+    (property "mpn" "CL21A475KLCLQNC" (at 64.516 159.512 0)
+      (effects (font (size 1.27 1.27)) hide)
+    )
     (pin "1")
     (pin "2")
@@
       (effects (font (size 1.27 1.27)) hide)
     )
+    (property "mpn" "CL32A106KAULNNE" (at 48.514 159.512 0)
+      (effects (font (size 1.27 1.27)) hide)
+    )
     (pin "1")
     (pin "2")
@@
       (effects (font (size 1.27 1.27)) hide)
     )
+    (property "mpn" "150060GS75000" (at 119.634 157.734 0)
+      (effects (font (size 1.27 1.27)) hide)
+    )
     (pin "1")
     (pin "2")
@@
       (effects (font (size 1.27 1.27)) hide)
     )
+    (property "mpn" "CL32A106KAULNNE" (at 101.6 158.75 0)
+      (effects (font (size 1.27 1.27)) hide)
+    )
     (pin "1")
     (pin "2")
@@
     )
     (property "Datasheet" "https://www.murata.com/en-us/products/productdata/8796739862558/ENFA0007.pdf" (at 135.636 75.946 0)
+      (effects (font (size 1.27 1.27)) hide)
+    )
+    (property "MouserPN" "81-BLM41P600S" (at 135.636 75.946 0)
+      (effects (font (size 1.27 1.27)) hide)
+    )
+    (property "mpn" "BLM41PG600SN1L" (at 135.636 75.946 0)
       (effects (font (size 1.27 1.27)) hide)
     )
@@
       (effects (font (size 1.27 1.27)) hide)
     )
+    (property "mpn" "150060GS75000" (at 154.686 79.756 0)
+      (effects (font (size 1.27 1.27)) hide)
+    )
     (pin "1")
     (pin "2")
@@
       (effects (font (size 1.27 1.27)) (justify left))
     )
-    (property "Footprint" "LaserBoardR5:C_0603_1608Metric_Pad1.08x0.95mm_HandSolder" (at 143.9672 91.948 0)
+    (property "Footprint" "LaserBoardR5:C_0603_1608Metric" (at 143.9672 91.948 0)
       (effects (font (size 1.27 1.27)) hide)
     )
@@
       (effects (font (size 1.27 1.27)) hide)
     )
+    (property "mpn" "C603C104K5RAC3121" (at 143.002 88.138 0)
+      (effects (font (size 1.27 1.27)) hide)
+    )

Commit message: Rev 5a
Parts:
- C15: footprint LaserBoardR5:CP_Elec_6.3x9.9 -> Capacitor_THT:CP_Radial_D6.3mm_P2.50mm
- R20, R21: MouserPN (none) -> 603-RC0603JR-0720KL; mpn (none) -> RC0603JR-0720KL
Changed lines of the file:
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@@
+      (effects (font (size 1.27 1.27)) hide)
+    )
+    (property "Notes" "" (at 126.238 87.884 0)
       (effects (font (size 1.27 1.27)) hide)
     )
@@
       (effects (font (size 1.27 1.27)) hide)
     )
+    (property "Notes" "" (at 78.74 94.234 0)
+      (effects (font (size 1.27 1.27)) hide)
+    )
     (pin "1")
     (pin "2")
@@
     )
     (property "Datasheet" "~" (at 119.634 166.878 0)
+      (effects (font (size 1.27 1.27)) hide)
+    )
+    (property "MouserPN" "603-RC0603JR-0720KL" (at 119.634 166.878 0)
+      (effects (font (size 1.27 1.27)) hide)
+    )
+    (property "Notes" "" (at 119.634 166.878 0)
+      (effects (font (size 1.27 1.27)) hide)
+    )
+    (property "mpn" "RC0603JR-0720KL" (at 119.634 166.878 0)
       (effects (font (size 1.27 1.27)) hide)
     )
@@
       (effects (font (size 1.27 1.27)) hide)
     )
+    (property "Notes" "" (at 83.82 133.096 0)
+      (effects (font (size 1.27 1.27)) hide)
+    )
     (pin "1")
     (pin "2")
@@
       (effects (font (size 1.27 1.27)) (justify left))
     )
-    (property "Footprint" "LaserBoardR5:CP_Elec_6.3x9.9" (at 168.3512 89.916 0)
+    (property "Footprint" "Capacitor_THT:CP_Radial_D6.3mm_P2.50mm" (at 168.3512 89.916 0)
       (effects (font (size 1.27 1.27)) hide)
     )
@@
       (effects (font (size 1.27 1.27)) hide)
     )
+    (property "Notes" "" (at 167.386 86.106 0)
+      (effects (font (size 1.27 1.27)) hide)
+    )
     (pin "1")
     (pin "2")
@@
       (effects (font (size 1.27 1.27)) hide)
     )
+    (property "Notes" "" (at 64.516 159.512 0)
+      (effects (font (size 1.27 1.27)) hide)
+    )
     (pin "1")
     (pin "2")
@@
       (effects (font (size 1.27 1.27)) hide)
     )
+    (property "Notes" "" (at 48.514 159.512 0)
+      (effects (font (size 1.27 1.27)) hide)
+    )
     (pin "1")
     (pin "2")
@@
       (effects (font (size 1.27 1.27)) hide)
     )
+    (property "Notes" "" (at 119.634 157.734 0)
+      (effects (font (size 1.27 1.27)) hide)
+    )
     (pin "1")
     (pin "2")
@@
       (effects (font (size 1.27 1.27)) hide)
     )
+    (property "MouserPN" "603-RC0603JR-0720KL" (at 154.686 88.9 0)
+      (effects (font (size 1.27 1.27)) hide)
+    )
+    (property "Notes" "" (at 154.686 88.9 0)
+      (effects (font (size 1.27 1.27)) hide)
+    )
+    (property "mpn" "RC0603JR-0720KL" (at 154.686 88.9 0)
+      (effects (font (size 1.27 1.27)) hide)
+    )
     (pin "1")
     (pin "2")
@@
       (effects (font (size 1.27 1.27)) hide)
     )
+    (property "Notes" "" (at 101.6 158.75 0)
+      (effects (font (size 1.27 1.27)) hide)
+    )
     (pin "1")
     (pin "2")
@@
       (effects (font (size 1.27 1.27)) hide)
     )
+    (property "Notes" "" (at 78.74 82.804 0)
+      (effects (font (size 1.27 1.27)) hide)
+    )
     (pin "1")
     (pin "2")
@@
     )
     (property "mpn" "BLM41PG600SN1L" (at 135.636 75.946 0)
+      (effects (font (size 1.27 1.27)) hide)
+    )
+    (property "Notes" "" (at 135.636 75.946 0)
       (effects (font (size 1.27 1.27)) hide)
     )
@@
       (effects (font (size 1.27 1.27)) hide)
     )
+    (property "Notes" "" (at 154.686 79.756 0)
+      (effects (font (size 1.27 1.27)) hide)
+    )
     (pin "1")
     (pin "2")
@@
     )
     (property "mpn" "SMAJ28CA" (at 110.998 87.122 0)
+      (effects (font (size 1.27 1.27)) hide)
+    )
+    (property "Notes" "" (at 110.998 87.122 0)
       (effects (font (size 1.27 1.27)) hide)
     )
@@
       (effects (font (size 1.27 1.27)) hide)
     )
+    (property "Notes" "" (at 102.108 80.264 0)
+      (effects (font (size 1.27 1.27)) hide)
+    )
     (pin "1")
     (pin "2")
@@
       (effects (font (size 1.27 1.27)) hide)
     )
+    (property "Notes" "" (at 143.002 88.138 0)
+      (effects (font (size 1.27 1.27)) hide)
+    )
